Commit message: laser scan matcher and dwa config

File: ired_bringup/urdf/robot.urdf.xacro (robot description, xacro)
@@ -1,4 +1,4 @@
 <?xml version="1.0"?>
-<robot name="IRED">
+<robot name="iRED Robot">
     <!-- link -->
     <link name="base_footprint"/>
@@ -11,10 +11,10 @@
         <parent link="base_footprint"/>
         <child link="base_link"/>
-        <origin xyz="0.0 0.0 0.0" rpy="0.0 0.0 0.0"/>
+        <origin xyz="0.0 0.0 0.08" rpy="0.0 0.0 0.0"/>
     </joint>
     <joint name="scan_joint" type="fixed">
         <parent link="base_link"/>
         <child link="base_scan"/>
-        <origin xyz="0.0 0.0 0.0" rpy="0.0 0.0 0.0"/>
+        <origin xyz="0.0 0.0 0.125" rpy="0.0 0.0 0.0"/>
     </joint>
     <joint name="wheel_right_joint" type="continuous">
@@ -22,5 +22,5 @@
         <child link="wheel_right_link"/>
         <axis xyz="0 0 1"/>
-        <origin xyz="0.0 0.0 0.0" rpy="0.0 0.0 0.0"/>
+        <origin xyz="0.0 -0.106 -0.04" rpy="-1.57 0.0 0.0"/>
     </joint>
     <joint name="wheel_left_joint" type="continuous">
@@ -28,5 +28,5 @@
         <child link="wheel_left_link"/>
         <axis xyz="0 0 1"/>
-        <origin xyz="0.0 0.0 0.0" rpy="0.0 0.0 0.0"/>
+        <origin xyz="0.0 0.106 -0.04" rpy="-1.57 0.0 0.0"/>
     </joint>
 </robot>
